Commit message: ddw

File: ROS Packages/amr_model/urdf/amr_model.urdf (robot description, URDF)
Before this commit: robot amr_model, 4 links, 3 joints
Links:
- removed link Link 3
- removed link Link_1
- removed link Link_2
- added link Back_Left_Castor_Link, mass 0.16139609361482; collision mesh filename=package://amr_model/meshes/Back_Left_Castor_Link.STL; visual mesh filename=package://amr_model/meshes/Back_Left_Castor_Link.STL
- added link Back_Left_Swivel_Link, mass 0.0403332300930945; collision mesh filename=package://amr_model/meshes/Back_Left_Swivel_Link.STL; visual mesh filename=package://amr_model/meshes/Back_Left_Swivel_Link.STL
- added link Back_Link, mass 0.241012788592428; collision mesh filename=package://amr_model/meshes/Back_Link.STL; visual mesh filename=package://amr_model/meshes/Back_Link.STL
- added link Back_RIght_Swivel_Link, mass 0.0403332394157405; collision mesh filename=package://amr_model/meshes/Back_RIght_Swivel_Link.STL; visual mesh filename=package://amr_model/meshes/Back_RIght_Swivel_Link.STL
- added link Back_Right_Castor_Link, mass 0.161396093614819; collision mesh filename=package://amr_model/meshes/Back_Right_Castor_Link.STL; visual mesh filename=package://amr_model/meshes/Back_Right_Castor_Link.STL
- added link Left_Castor_Link, mass 0.16139609361482; collision mesh filename=package://amr_model/meshes/Left_Castor_Link.STL; visual mesh filename=package://amr_model/meshes/Left_Castor_Link.STL
- added link Left_Drive_Link, mass 0.697781408700204; collision mesh filename=package://amr_model/meshes/Left_Drive_Link.STL; visual mesh filename=package://amr_model/meshes/Left_Drive_Link.STL
- added link Left_Link, mass 0.173725014087237; collision mesh filename=package://amr_model/meshes/Left_Link.STL; visual mesh filename=package://amr_model/meshes/Left_Link.STL
- added link Left_Swivel_Link, mass 0.040333223205091; collision mesh filename=package://amr_model/meshes/Left_Swivel_Link.STL; visual mesh filename=package://amr_model/meshes/Left_Swivel_Link.STL
- added link Right_Castor_Link, mass 0.161396093614819; collision mesh filename=package://amr_model/meshes/Right_Castor_Link.STL; visual mesh filename=package://amr_model/meshes/Right_Castor_Link.STL
- added link Right_Drive_Link, mass 0.697781408700203; collision mesh filename=package://amr_model/meshes/Right_Drive_Link.STL; visual mesh filename=package://amr_model/meshes/Right_Drive_Link.STL
- added link Right_Link, mass 0.173725014087434; collision mesh filename=package://amr_model/meshes/Right_Link.STL; visual mesh filename=package://amr_model/meshes/Right_Link.STL
- added link Right_Swivel_Link, mass 0.0403332244174408; collision mesh filename=package://amr_model/meshes/Right_Swivel_Link.STL; visual mesh filename=package://amr_model/meshes/Right_Swivel_Link.STL
- link base_link: mass 3.93344073192101 -> 3.76763445588817
Joints:
- removed joint back_pivot
- removed joint left_pivot
- removed joint right_pivot
- added joint Back_Joint: type continuous, parent base_link, child Back_Link, origin xyz=-0.24999 0 0.052812 rpy=0 1.5708 0, axis 0 0 1
- added joint Back_Left_Castor_Joint: type continuous, parent Back_Left_Swivel_Link, child Back_Left_Castor_Link, origin xyz=0.042 0 0.0755 rpy=1.5708 -0.060395 0, axis 0 0 1
- added joint Back_Left_Swivel_Joint: type continuous, parent Back_Link, child Back_Left_Swivel_Link, origin xyz=0 0.1605 0.0005 rpy=-1.5708 -1.5673 -1.5708, axis 0 0 -1
- added joint Back_RIght_Swivel_Joint: type continuous, parent Back_Link, child Back_RIght_Swivel_Link, origin xyz=0 -0.1605 0.0005 rpy=1.5708 0 1.5708, axis 0 0 -1
- added joint Back_Right_Castor_Joint: type continuous, parent Back_RIght_Swivel_Link, child Back_Right_Castor_Link, origin xyz=0.00036509 0.041998 0.0755 rpy=1.5708 0.3931 1.5621, axis 0 0 1
- added joint Left_Castor_Joint: type continuous, parent Left_Swivel_Link, child Left_Castor_Link, origin xyz=-0.042008 0 0.075496 rpy=-1.5708 0.00010282 0.00010282, axis 0 0 1
- added joint Left_Drive_Joint: type continuous, parent Left_Link, child Left_Drive_Link, origin xyz=-0.12751 0.050237 0.0546 rpy=0 0 0, axis 0 0 -1
- added joint Left_Joint: type continuous, parent base_link, child Left_Link, origin xyz=0.12751 0.1625 0.052812 rpy=-1.5708 0 0, axis 0 0 1
- added joint Left_Swivel_Joint: type continuous, parent Left_Link, child Left_Swivel_Link, origin xyz=0.123 1.2647E-05 -0.0005 rpy=-1.5708 0 0, axis 0.00010282 0 -1
- added joint Right_Castor_Joint: type continuous, parent Right_Swivel_Link, child Right_Castor_Link, origin xyz=0 -0.041993 0.075504 rpy=0 1.5708 0, axis 0 9.054E-05 -1
- added joint Right_Drive_Joint: type continuous, parent Right_Link, child Right_Drive_Link, origin xyz=0.1275 0.050262 0.055649 rpy=0 0 0, axis 0 0 -1
- added joint Right_Joint: type continuous, parent base_link, child Right_Link, origin xyz=0.12751 -0.1625 0.052812 rpy=-1.5708 0 3.1416, axis 0 0 -1
- added joint Right_Swivel_Joint: type continuous, parent Right_Link, child Right_Swivel_Link, origin xyz=-0.123 -1.1136E-05 0.0005 rpy=1.5708 1.5708 0, axis 0 -9.054E-05 -1
