Commit message: dwd

File: ROS Packages/amr_model_2/urdf/amr_model_2.urdf (robot description, URDF)
Before this commit: robot amr_model, 14 links, 13 joints
Links:
- link Back_Left_Castor_Link: geometry collision mesh filename=package://amr_model_2/meshes/Back_Left_Castor_Link.STL; visual mesh filename=package://amr_model_2/meshes/Back_Left_Castor_Link.STL
- link Back_Left_Swivel_Link: geometry collision mesh filename=package://amr_model_2/meshes/Back_Left_Swivel_Link.STL; visual mesh filename=package://amr_model_2/meshes/Back_Left_Swivel_Link.STL
- link Back_Link: geometry collision mesh filename=package://amr_model_2/meshes/Back_Link.STL; visual mesh filename=package://amr_model_2/meshes/Back_Link.STL
- link Back_RIght_Swivel_Link: geometry collision mesh filename=package://amr_model_2/meshes/Back_RIght_Swivel_Link.STL; visual mesh filename=package://amr_model_2/meshes/Back_RIght_Swivel_Link.STL
- link Back_Right_Castor_Link: geometry collision mesh filename=package://amr_model_2/meshes/Back_Right_Castor_Link.STL; visual mesh filename=package://amr_model_2/meshes/Back_Right_Castor_Link.STL
- link Left_Castor_Link: geometry collision mesh filename=package://amr_model_2/meshes/Left_Castor_Link.STL; visual mesh filename=package://amr_model_2/meshes/Left_Castor_Link.STL
- link Left_Drive_Link: geometry collision mesh filename=package://amr_model_2/meshes/Left_Drive_Link.STL; visual mesh filename=package://amr_model_2/meshes/Left_Drive_Link.STL
- link Left_Link: geometry collision mesh filename=package://amr_model_2/meshes/Left_Link.STL; visual mesh filename=package://amr_model_2/meshes/Left_Link.STL
- link Left_Swivel_Link: geometry collision mesh filename=package://amr_model_2/meshes/Left_Swivel_Link.STL; visual mesh filename=package://amr_model_2/meshes/Left_Swivel_Link.STL
- link Right_Castor_Link: mass 0.161396093614819 -> 0.161396093614818; geometry collision mesh filename=package://amr_model_2/meshes/Right_Castor_Link.STL; visual mesh filename=package://amr_model_2/meshes/Right_Castor_Link.STL
- link Right_Drive_Link: geometry collision mesh filename=package://amr_model_2/meshes/Right_Drive_Link.STL; visual mesh filename=package://amr_model_2/meshes/Right_Drive_Link.STL
- link Right_Link: geometry collision mesh filename=package://amr_model_2/meshes/Right_Link.STL; visual mesh filename=package://amr_model_2/meshes/Right_Link.STL
- link Right_Swivel_Link: mass 0.0403332244174408 -> 0.0403332724407856; geometry collision mesh filename=package://amr_model_2/meshes/Right_Swivel_Link.STL; visual mesh filename=package://amr_model_2/meshes/Right_Swivel_Link.STL
- link base_link: geometry collision mesh filename=package://amr_model_2/meshes/base_link.STL; visual mesh filename=package://amr_model_2/meshes/base_link.STL
Joints:
- joint Back_Joint: origin xyz=-0.24999 0 0.052812 rpy=0 1.5708 0 -> xyz=-0.249993740776166 0 0.0528119631753474 rpy=0 1.5707963267949 0
- joint Left_Castor_Joint: origin xyz=-0.042008 0 0.075496 rpy=-1.5708 0.00010282 0.00010282 -> xyz=-0.042008 0 0.075496 rpy=0 0 0
- joint Left_Joint: origin xyz=0.12751 0.1625 0.052812 rpy=-1.5708 0 0 -> xyz=0.12751 0.1625 0.052812 rpy=0 0 0
- joint Left_Swivel_Joint: origin xyz=0.123 1.2647E-05 -0.0005 rpy=-1.5708 0 0 -> xyz=0.123 1.2647E-05 -0.0005 rpy=0 0 0
- joint Right_Castor_Joint: origin xyz=0 -0.041993 0.075504 rpy=0 1.5708 0 -> xyz=0 -0.041993 0.075504 rpy=0 0 0
- joint Right_Joint: origin xyz=0.12751 -0.1625 0.052812 rpy=-1.5708 0 3.1416 -> xyz=0.127506259223797 -0.162500000000007 0.0528119631753412 rpy=-1.5707963267949 0 3.14159265358979
- joint Right_Swivel_Joint: axis 0 -9.054E-05 -1 -> 0 -9.05402263184918E-05 -0.999999995901234; origin xyz=-0.123 -1.1136E-05 0.0005 rpy=1.5708 1.5708 0 -> xyz=-0.122999999495851 -1.11364478370679E-05 0.000500000000000833 rpy=1.5707963267949 1.5707963267949 0
