Commit message: ll

File: Models/basic_amr/URDF/basic_amr/urdf/basic_amr.urdf (robot description, URDF)
Before this commit: robot basic_amr, 11 links, 10 joints
Links:
- link base_link: mass 4.4522 -> 4.45218985232546
- link castor_BR_swivel: mass 0 -> 0.0403332436496892
- link castor_BR_wheel: mass 0.161396093614819 -> 0.16139609361482
- link castor_FL_swivel: mass 0.040333 -> 0.0403332267042345
- link left_wheel: mass 0.67187 -> 0.671865219229546
- link right_wheel: mass 0.67187 -> 0.671865219229547
Joints:
- joint castor_BL_swivel_hinge: origin xyz=-0.1605 -0.2495 0.0595 rpy=0 0 0.0024111 -> xyz=-0.160500000000001 -0.249499999999981 0.0595000000000003 rpy=0 0 0.00241105480749667
- joint castor_BL_wheel_hinge: axis -0.0024111 0 -1 -> -0.00241105247151348 0 -0.999997093408766; origin xyz=-0.001 -0.042 -0.0845 rpy=1.5708 0 1.5684 -> xyz=-0.00100000000000017 -0.0419999999999998 -0.0845 rpy=1.5707963267949 0 1.5683852719874
- joint castor_BR_swivel_hinge: origin xyz=0.1605 -0.2495 0.0595 rpy=0 0 0.010886 -> xyz=0.160499999999999 -0.249499999999981 0.0594999999999991 rpy=0 0 0.0108863057088858
- joint castor_BR_wheel_hinge: axis 0.010886 0 0.99994 -> 0.0108860906844809 0 0.999940744759213; origin xyz=0.001 -0.042 -0.0845 rpy=1.5708 0 1.5599 -> xyz=0.000999999999999751 -0.0419999999999998 -0.0845 rpy=1.5707963267949 0 1.55991002108601
- joint castor_FL_swivel_hinge: origin xyz=-0.162 0.2505 0.0595 rpy=0 0 -0.0016249 -> xyz=-0.161999999999996 0.250499999999998 0.0595000000000003 rpy=0 0 -0.00162492292127055
- joint castor_FL_wheel_hinge: axis 0.0016249 0 -1 -> 0.00162492220620229 0 -0.99999867981304; origin xyz=-0.001 -0.042 -0.0845 rpy=1.5708 0 1.5724 -> xyz=-0.000999999999999973 -0.042 -0.0845 rpy=1.5707963267949 0 1.57242124971617
- joint castor_FR_swivel_hinge: origin xyz=0.163 0.2505 0.0595 rpy=0 0 0 -> xyz=0.163000000000007 0.250500000000009 0.0594999999999989 rpy=0 0 0
- joint left_wheel_hinge: origin xyz=-0.2231 0 0.00025 rpy=0 0 0 -> xyz=-0.223099999999995 0 0.00024999999999966 rpy=1.5707963267949 0 1.5707963267949
- joint right_wheel_hinge: origin xyz=0.2231 0 0.00025 rpy=0 0 0 -> xyz=0.223100000000009 0 0.000249999999998834 rpy=1.5707963267949 0 1.5707963267949

Commit message: hi

File: Models/basic_amr/URDF/basic_amr/urdf/basic_amr.urdf (robot description, URDF)
Before this commit: robot basic_amr, 11 links, 10 joints
Links:
- removed link castor_BL_swivel
- removed link castor_BL_wheel
- removed link castor_BR_swivel
- removed link castor_BR_wheel
- removed link castor_FL_swivel
- removed link castor_FL_wheel
- removed link castor_FR_swivel
- removed link castor_FR_wheel
- added link castor_BL, mass 0.161396093614819; collision mesh filename=package://basic_amr/meshes/castor_BL.STL; visual mesh filename=package://basic_amr/meshes/castor_BL.STL
- added link castor_BR, mass 0.161396093614819; collision mesh filename=package://basic_amr/meshes/castor_BR.STL; visual mesh filename=package://basic_amr/meshes/castor_BR.STL
- added link castor_FL, mass 0.16139609361482; collision mesh filename=package://basic_amr/meshes/castor_FL.STL; visual mesh filename=package://basic_amr/meshes/castor_FL.STL
- added link castor_FR, mass 0.161396093614819; collision mesh filename=package://basic_amr/meshes/castor_FR.STL; visual mesh filename=package://basic_amr/meshes/castor_FR.STL
- added link swivel_BL, mass 0; collision mesh filename=package://basic_amr/meshes/swivel_BL.STL; visual mesh filename=package://basic_amr/meshes/swivel_BL.STL
- added link swivel_BR, mass 0.0401879953591256; collision mesh filename=package://basic_amr/meshes/swivel_BR.STL; visual mesh filename=package://basic_amr/meshes/swivel_BR.STL
- added link swivel_FL, mass 0.0401879953591256; collision mesh filename=package://basic_amr/meshes/swivel_FL.STL; visual mesh filename=package://basic_amr/meshes/swivel_FL.STL
- added link swivel_FR, mass 0.0401879953591251; collision mesh filename=package://basic_amr/meshes/swivel_FR.STL; visual mesh filename=package://basic_amr/meshes/swivel_FR.STL
- link base_link: mass 4.45218985232546 -> 4.4522
Joints:
- removed joint castor_BL_swivel_hinge
- removed joint castor_BL_wheel_hinge
- removed joint castor_BR_swivel_hinge
- removed joint castor_BR_wheel_hinge
- removed joint castor_FL_swivel_hinge
- removed joint castor_FL_wheel_hinge
- removed joint castor_FR_swivel_hinge
- removed joint castor_FR_wheel_hinge
- added joint castor_BL_hinge: type continuous, parent swivel_BL, child castor_BL, origin xyz=-0.001 -0.042038 -0.081558 rpy=1.5708 0 1.5708, axis 0 0 -1
- added joint castor_BR_hinge: type continuous, parent swivel_BR, child castor_BR, origin xyz=0.001 -0.042038 -0.081558 rpy=1.5708 0 1.5708, axis 0 0 1
- added joint castor_FL_hinge: type continuous, parent swivel_FL, child castor_FL, origin xyz=0.001 -0.042038 -0.081558 rpy=1.5708 0 1.5708, axis 0 0 1
- added joint castor_FR_hinge: type continuous, parent swivel_FR, child castor_FR, origin xyz=0.001 -0.042038 -0.081558 rpy=1.5708 0 1.5708, axis 0 0 1
- added joint swivel_BL_hinge: type continuous, parent base_link, child swivel_BL, origin xyz=-0.1605 -0.2495 -0.072 rpy=0 0 0, axis 0 0 1
- added joint swivel_BR_hinge: type continuous, parent base_link, child swivel_BR, origin xyz=0.1605 -0.2495 -0.072 rpy=0 0 0, axis 0 0 1
- added joint swivel_FL_hinge: type continuous, parent base_link, child swivel_FL, origin xyz=-0.162 0.2505 -0.072 rpy=0 0 0, axis 0 0 1
- added joint swivel_FR_hinge: type continuous, parent base_link, child swivel_FR, origin xyz=0.163 0.2505 -0.072 rpy=0 0 0, axis 0 0 1
- joint left_wheel_hinge: axis 0 0 1 -> 0 0 -1; origin xyz=-0.223099999999995 0 0.00024999999999966 rpy=1.5707963267949 0 1.5707963267949 -> xyz=-0.2231 0 -0.13125 rpy=3.1416 -1.5708 0
- joint right_wheel_hinge: origin xyz=0.223100000000009 0 0.000249999999998834 rpy=1.5707963267949 0 1.5707963267949 -> xyz=0.2231 0 -0.13125 rpy=1.5708 0 1.5708

Commit message: new

File: Models/basic_amr/URDF/basic_amr/urdf/basic_amr.urdf (robot description, URDF)
Before this commit: robot basic_amr, 11 links, 10 joints
Links:
- link base_link: mass 4.4522 -> 4.45218985232546
- link swivel_BL: mass 0 -> 0.0401879953591248
Joints:
- joint castor_FR_hinge: origin xyz=0.001 -0.042038 -0.081558 rpy=1.5708 0 1.5708 -> xyz=0.00100000000000061 -0.0420375051343131 -0.0815575197240634 rpy=1.5707963267949 0 1.5707963267949

Commit message: plbo

File: Models/basic_amr/URDF/basic_amr/urdf/basic_amr.urdf (robot description, URDF)
Before this commit: robot basic_amr, 11 links, 10 joints
Links:
- link castor_BR: mass 0.161396093614819 -> 0.16139609361482
- link castor_FR: mass 0.161396093614819 -> 0.16139609361482
Joints:
- joint castor_BL_hinge: origin xyz=-0.001 -0.042038 -0.081558 rpy=1.5708 0 1.5708 -> xyz=-0.00100000000000036 -0.0420254389561341 -0.0825575197240612 rpy=1.5707963267949 0 1.5707963267949
- joint castor_BR_hinge: origin xyz=0.001 -0.042038 -0.081558 rpy=1.5708 0 1.5708 -> xyz=0.000999999999999668 -0.0420254389561336 -0.0825575197240624 rpy=1.5707963267949 0 1.5707963267949
- joint castor_FL_hinge: origin xyz=0.001 -0.042038 -0.081558 rpy=1.5708 0 1.5708 -> xyz=0.000999999999999168 -0.042025438956134 -0.0825575197240596 rpy=1.5707963267949 0 1.5707963267949
- joint castor_FR_hinge: origin xyz=0.00100000000000061 -0.0420375051343131 -0.0815575197240634 rpy=1.5707963267949 0 1.5707963267949 -> xyz=0.00100000000000061 -0.0420254389561369 -0.0825575197240634 rpy=1.5707963267949 0 1.5707963267949
- joint left_wheel_hinge: origin xyz=-0.2231 0 -0.13125 rpy=3.1416 -1.5708 0 -> xyz=-0.223099999999996 0 -0.13125 rpy=3.14159265358979 -1.5707963267949 0
- joint right_wheel_hinge: origin xyz=0.2231 0 -0.13125 rpy=1.5708 0 1.5708 -> xyz=0.223100000000008 0 -0.131250000000001 rpy=1.5707963267949 0 1.5707963267949
- joint swivel_BL_hinge: origin xyz=-0.1605 -0.2495 -0.072 rpy=0 0 0 -> xyz=-0.160500000000002 -0.249499999999982 -0.0719999999999989 rpy=0 0 0
- joint swivel_BR_hinge: origin xyz=0.1605 -0.2495 -0.072 rpy=0 0 0 -> xyz=0.160499999999998 -0.249499999999981 -0.0719999999999989 rpy=0 0 0
- joint swivel_FL_hinge: origin xyz=-0.162 0.2505 -0.072 rpy=0 0 0 -> xyz=-0.161999999999997 0.250499999999997 -0.0720000000000005 rpy=0 0 0
- joint swivel_FR_hinge: origin xyz=0.163 0.2505 -0.072 rpy=0 0 0 -> xyz=0.163000000000006 0.250500000000009 -0.0720000000000007 rpy=0 0 0
