Commit message: colour

File: Models/full_amr/URDF/full_amr/urdf/full_amr.urdf (robot description, URDF)
Before this commit: robot full_amr, 14 links, 13 joints
Links:
- link FR_castor: mass 0.161396093614819 -> 0.16139609361482
- link FR_swivel: mass 0.0403332237188925 -> 0.0403331792084209
- link back_pivot: mass 0.241012788592428 -> 0.24101
- link base_link: mass 3.86321584157732 -> 3.8632
- link left_pivot: mass 0.173980611061865 -> 0.17398
- link right_pivot: mass 0.173980611077858 -> 0.17398
- link right_wheel: mass 0.671865219229547 -> 0.671865219229546
Joints:
- joint FR_castor_hinge: origin xyz=0.00100000000000031 -0.0420000000000006 -0.0845000000000024 rpy=0 0 0 -> xyz=0.00099999999997849 -0.0425510539838774 -0.0842238553194065 rpy=0 0 0
- joint FR_swivel_hinge: axis 0 0 1 -> 0 0.00653195251969943 0.999978666570583; origin xyz=0.000499999999998585 0.123000000000001 0.00900000000000202 rpy=0 0 0 -> xyz=0.000499999999999584 0.123056163560861 0.00819637783921516 rpy=0 0 0
- joint back_pivot_hinge: origin xyz=0 -0.25 -0.081 rpy=0 0 0 -> xyz=0 -0.24999999999999 -0.0810000000000002 rpy=0 0 0
- joint left_pivot_hinge: origin xyz=-0.1625 0.1275 -0.081 rpy=0 0 0 -> xyz=-0.162500000000001 0.12749999999999 -0.081 rpy=0 0 0
- joint right_pivot_hinge: origin xyz=0.1625 0.1275 -0.081 rpy=0 0 0 -> xyz=0.162500000000008 0.127500000000012 -0.0809999999999999 rpy=0 0 0
- joint right_wheel_hinge: origin xyz=0.0606000000000009 -0.127499999999999 -0.0502500000000001 rpy=1.5707963267949 0 1.5707963267949 -> xyz=0.060600000000002 -0.127825510601864 -0.0494161040489112 rpy=1.5707963267949 0 1.5707963267949
