Commit message: jj

File: Models/full_amr_sensor/urdf/full_amr_sensor.urdf (robot description, URDF)
Before this commit: robot full_amr_sensor, 17 links, 16 joints
Links:
- link back_pivot: mass 0.241012788592429 -> 0.241012788592428
- link right_wheel: mass 0.671865219229547 -> 0.671865219229546
- link zed2: mass 0.152262285698166 -> 0.152262285698153
Joints:
- joint m2m2_hinge: origin xyz=-0.0073926 0.32076 -0.061 rpy=0 0 0 -> xyz=-0.00499999999999948 0.3075 -0.0609999999999998 rpy=0 0 -1.57079632679489
- joint zed2_hinge: origin xyz=-0.081402 0.37212 -0.090184 rpy=0 0 1.5708 -> xyz=-0.0599999999999997 0.37395326786623 -0.0901838222464366 rpy=0 0 1.5707963267949
