Commit message: eee

File: Models/full_amr/URDF/Raw/full_amr/urdf/full_amr.urdf (robot description, URDF)
Before this commit: robot full_amr, 14 links, 13 joints
Links:
- added link imu, mass 0; collision mesh filename=package://full_amr/meshes/imu.STL; visual mesh filename=package://full_amr/meshes/imu.STL
- added link m2m2, mass 0.19138; collision mesh filename=package://full_amr/meshes/m2m2.STL; visual mesh filename=package://full_amr/meshes/m2m2.STL
- added link zed2, mass 0.15226; collision mesh filename=package://full_amr/meshes/zed2.STL; visual mesh filename=package://full_amr/meshes/zed2.STL
- link BL_castor: mass 0.16139609361482 -> 0.1614
- link BL_swivel: mass 0.040333232832404 -> 0.040333
- link BR_castor: mass 0.16139609361482 -> 0.1614
- link BR_swivel: mass 0.0403332273268806 -> 0.040333
- link FL_castor: mass 0.161396093614819 -> 0.1614
- link FL_swivel: mass 0.0403332363730702 -> 0.040333
- link FR_castor: mass 0.16139609361482 -> 0.1614
- link FR_swivel: mass 0.0403331792084209 -> 0.040333
- link back_pivot: mass 0.24101 -> 0.241012788592429
- link left_wheel: mass 0.671865219229547 -> 0.67187
- link right_wheel: mass 0.671865219229546 -> 0.67187
Joints:
- added joint imu_hinge: type fixed, parent base_link, child imu, origin xyz=0 0.2275 -0.0980997999999998 rpy=3.14159265358979 0 0, axis 0 0 0
- added joint m2m2_hinge: type fixed, parent base_link, child m2m2, origin xyz=-0.005 0.3075 -0.061 rpy=0 0 -1.5708, axis 0 0 0
- added joint zed2_hinge: type fixed, parent base_link, child zed2, origin xyz=-0.06 0.37395 -0.090184 rpy=0 0 1.5708, axis 0 0 0
- joint back_pivot_hinge: origin xyz=0 -0.24999999999999 -0.0810000000000002 rpy=0 0 0 -> xyz=0 -0.25 -0.081 rpy=0 0 0
- joint left_pivot_hinge: origin xyz=-0.162500000000001 0.12749999999999 -0.081 rpy=0 0 0 -> xyz=-0.1625 0.1275 -0.081 rpy=0 0 0
- joint right_pivot_hinge: origin xyz=0.162500000000008 0.127500000000012 -0.0809999999999999 rpy=0 0 0 -> xyz=0.1625 0.1275 -0.081 rpy=0 0 0
- joint right_wheel_hinge: origin xyz=0.060600000000002 -0.127825510601864 -0.0494161040489112 rpy=1.5707963267949 0 1.5707963267949 -> xyz=0.0606 -0.12783 -0.049416 rpy=1.5708 0 1.5708
