Commit message: dd

File: ROS Packages/full_amr_sensor/urdf/full_amr_sensor.urdf (robot description, URDF)
Before this commit: robot full_amr_sensor, 17 links, 16 joints
Links:
- removed link zed2
- added link zed2_base_link, mass 0.152262285698166; collision mesh filename=package://full_amr_sensor/meshes/zed2.STL; visual mesh filename=package://full_amr_sensor/meshes/zed2.STL
Joints:
- joint zed2_hinge: child zed2 -> zed2_base_link

Commit message: ddd

File: ROS Packages/full_amr_sensor/urdf/full_amr_sensor.urdf (robot description, URDF)
Before this commit: robot full_amr_sensor, 17 links, 16 joints
Links:
- removed link m2m2
- added link laser, mass 0.191381897465873; collision mesh filename=package://full_amr_sensor/meshes/m2m2.STL; visual mesh filename=package://full_amr_sensor/meshes/m2m2.STL
Joints:
- joint m2m2_hinge: child m2m2 -> laser

Commit message: ddd

File: ROS Packages/full_amr_sensor/urdf/full_amr_sensor.urdf (robot description, URDF)
Before this commit: robot full_amr_sensor, 17 links, 16 joints
Links:
- removed link laser
- added link m2m2, mass 0.191381897465873; collision mesh filename=package://full_amr_sensor/meshes/m2m2.STL; visual mesh filename=package://full_amr_sensor/meshes/m2m2.STL
Joints:
- joint m2m2_hinge: child laser -> m2m2

Commit message: ddd

File: ROS Packages/full_amr_sensor/urdf/full_amr_sensor.urdf (robot description, URDF)
Before this commit: robot full_amr_sensor, 17 links, 16 joints
Links:
- removed link zed2_base_link
- added link zed2, mass 0.152262285698166; collision mesh filename=package://full_amr_sensor/meshes/zed2.STL; visual mesh filename=package://full_amr_sensor/meshes/zed2.STL
Joints:
- joint zed2_hinge: child zed2_base_link -> zed2
