Commit message: ddwdw

File: ROS Packages/full_amr_sensor/urdf/full_amr_sensor0.urdf (robot description, URDF)
Before this commit: robot full_amr_sensor, 17 links, 16 joints
Links:
- removed link base_link_true
- added link m2m2, mass 0.191381897465873; collision mesh filename=package://full_amr_sensor/meshes/m2m2.STL; visual mesh filename=package://full_amr_sensor/meshes/m2m2.STL
- link base_link: mass 0.191381897465873 -> 3.86321584157732; geometry collision mesh filename=package://full_amr_sensor/meshes/base_link.STL; visual mesh filename=package://full_amr_sensor/meshes/base_link.STL
Joints:
- joint back_pivot_hinge: parent base_link_true -> base_link
- joint imu_hinge: parent base_link_true -> base_link
- joint left_pivot_hinge: parent base_link_true -> base_link
- joint m2m2_hinge: child base_link -> m2m2; parent base_link_true -> base_link
- joint right_pivot_hinge: parent base_link_true -> base_link
- joint zed2_hinge: parent base_link_true -> base_link
